Commit message: update urdf xacro

File: thesis_robot/urdf/materials.xacro (robot description, xacro)
@@ -17,5 +17,5 @@
   </material>
   <material name="brown">
-    <color rgba="${222/255} ${207/255} ${195/255} 1.0"/>
+    <color rgba="0.87 0.82 0.76 1.0"/>
   </material>
   <material name="red">

File: thesis_robot/urdf/thesis_robot.urdf.xacro (robot description, xacro)
@@ -1,3 +1,2 @@
-<!-- <?xml version="1.0" encoding="UTF-8"?> -->
 <?xml version="1.0"?>
 <robot name="thesis_robot" xmlns:xacro="http://ros.org/wiki/xacro">
@@ -33,6 +32,12 @@
         #########
  -->
+  <!-- link gốc sẽ ko có joint  -->
+  <link name="base_footprint"/>
+  <joint name="base_joint" type="fixed">
+    <parent link="base_footprint"/>
+    <child link="base_link"/>
+    <origin xyz="0.0 0.0 0.0" rpy="0 0 0"/>
+  </joint>
 <!-- Base Link -->
-<!-- link gốc sẽ ko có joint  -->
 <!-- Vì ko đặt riêng link = "base_footprint" nên mọi mô tả (geometry) đều được tính từ tâm [0,0,0] theo cả 3 chiều nên khi tính độ cao phải chia /2 -->
   <link name="base_link">
@@ -77,5 +82,5 @@
      <!-- Tam phia tren cung -->
     <visual name="base_level2">
-      <origin xyz="0 0 0.325" rpy="0 0 0" />
+      <origin xyz="0 0 0.325" rpy="0 0 0" /> <!--125+200=325cm-->
       <geometry>
           <box size="0.3757 0.280 0.003"/> <!-- Tấm Nhôm AL = 3mm -->
@@ -148,4 +153,10 @@
       </geometry>
     </collision>
+    <inertial>
+			<mass value="0.1"/>
+			<origin xyz="0 0 0"/>
+			<inertia ixx="0.012411765597" ixy="-0.000711733678" ixz="0.00050272983"
+				 iyy="0.015218160428" iyz="-0.000004273467" izz="0.011763977943"/>
+  	</inertial>
   </link>
   <!-- Các khớp (join) có kiểu: type="continuous" cần được pub lên (sensor_msgs::JointState) -->
@@ -153,5 +164,5 @@
     <parent link="base_link"/>
     <child link="wheel_left_link"/>
-    <origin xyz="-0.12535 0.16 0.0625" rpy="0 0 0" />
+    <origin xyz="-0.12535 0.165 0.0625" rpy="0 0 0" /> <!--0.16+0.005-->
     <axis xyz="0 1 0" />
   </joint>
@@ -173,4 +184,10 @@
       </geometry>
     </collision>
+    <inertial>
+			<mass value="0.1"/>
+			<origin xyz="0 0 0"/>
+			<inertia ixx="0.012411765597" ixy="-0.000711733678" ixz="0.00050272983"
+				 iyy="0.015218160428" iyz="-0.000004273467" izz="0.011763977943"/>
+  	</inertial>
   </link>
   <!-- Các khớp (join) có kiểu: type="continuous" cần được pub lên (sensor_msgs::JointState) -->
@@ -178,5 +195,5 @@
     <parent link="base_link"/>
     <child link="wheel_right_link"/>
-    <origin xyz="-0.12535 -0.16 0.0625" rpy="0 0 0" />
+    <origin xyz="-0.12535 -0.165 0.0625" rpy="0 0 0" />
     <axis xyz="0 1 0" />
   </joint>
