Commit message: update urdf && xacro

File: thesis_robot/urdf/thesis_robot.gazebo.xacro (robot description, xacro)
@@ -1,4 +1,4 @@
 <?xml version="1.0"?>
-<robot name="thesis_robot" xmlns:xacro="http://ros.org/wiki/xacro">
+<robot name="thesis_robot_sim" xmlns:xacro="http://ros.org/wiki/xacro">
   <xacro:arg name="laser_visual" default="false"/>
   <xacro:arg name="imu_visual"   default="false"/>
@@ -6,7 +6,4 @@
     <material>Gazebo/Blue</material>
   </gazebo>
-  <!-- <gazebo reference="left_wheel">
-    <material>Gazebo/Blue</material>
-  </gazebo> -->
   <gazebo reference="wheel_left_link">
     <mu1>0.1</mu1>
@@ -19,7 +16,4 @@
     <material>Gazebo/Black</material>
   </gazebo>
-  <!-- <gazebo reference="right_wheel">
-    <material>Gazebo/Blue</material>
-  </gazebo> -->
   <gazebo reference="wheel_right_link">
     <mu1>0.1</mu1>
@@ -39,7 +33,6 @@
     <material>Gazebo/FlatBlack</material>
   </gazebo>
-  <!-- Plugin : Dieu khien Robot loai: differential_drive_controller -->
-  <gazebo>
-    <plugin name="differential_drive_controller" filename="libgazebo_ros_diff_drive.so">
+   <gazebo>
+    <plugin name="thesis_drive_controller" filename="libgazebo_ros_diff_drive.so">
       <commandTopic>cmd_vel</commandTopic>
       <odometryTopic>odom</odometryTopic>
@@ -47,5 +40,5 @@
       <odometrySource>world</odometrySource>
       <publishOdomTF>true</publishOdomTF>
-      <robotBaseFrame>base_link</robotBaseFrame>
+      <robotBaseFrame>base_footprint</robotBaseFrame>
       <publishWheelTF>false</publishWheelTF>
       <publishTf>true</publishTf>
@@ -62,6 +55,5 @@
     </plugin>
   </gazebo>
-  <!-- Plugin: IMU -->
-  <!-- <gazebo>
+  <gazebo>
     <plugin name="imu_plugin" filename="libgazebo_ros_imu.so">
       <alwaysOn>true</alwaysOn>
@@ -91,7 +83,6 @@
     </plugin>
   </gazebo>
-   -->
   <!-- Plugin: Lidar -->
-  <!-- <gazebo reference="base_scan">
+  <gazebo reference="base_scan">
     <material>Gazebo/FlatBlack</material>
     <sensor type="ray" name="lds_lfcd_sensor">
@@ -124,4 +115,4 @@
       </plugin>
     </sensor>
-  </gazebo> -->
+  </gazebo>
 </robot>
